Commit message: Implement simple line urdf for testing

File: urdf/line.urdf (robot description, URDF)
Before this commit: robot myfirst, 1 links, 0 joints
Links:
- added link link1
- added link link2
- link base_link: geometry 
Joints:
- added joint joint1: type continuous, parent base_link, child link1, origin xyz=2 0 0 rpy=0 0 0, axis 0 1 0
- added joint joint2: type continuous, parent link1, child link2, origin xyz=2 0 0 rpy=0 0 0, axis 1 0 0

Commit message: Add LineJointStatePublisher

File: urdf/line.urdf (robot description, URDF)
Before this commit: robot myfirst, 3 links, 2 joints
Links:
- removed link link2
- link base_link: geometry visual cylinder length=2 radius=0.1
- link link1: geometry visual cylinder length=2 radius=0.1
Joints:
- removed joint joint2
- joint joint1: axis 0 1 0 -> 0 0 1; origin xyz=2 0 0 rpy=0 0 0 -> xyz=2 0 0 rpy=0 0 -1.57
